Commit message: work gazebo and nav2

File: telerobot_description/urdf/controllers/omni_drive.urdf.xacro (robot description, xacro)
@@ -2,17 +2,26 @@
   <xacro:macro name="omni_drive_controller">
     <gazebo>
-    <plugin name="object_controller" filename="libgazebo_ros_planar_move.so">
-      <ros>
-        <argument>odom:=odom/unfiltered</argument>
-      </ros>
-      <command_topic>cmd_vel</command_topic>
-      <odometry_topic>odom/unfiltered</odometry_topic>
-      <odometry_frame>odom</odometry_frame>
-      <odometry_rate>20.0</odometry_rate>
-      <robot_base_frame>base_footprint</robot_base_frame>
-      <publish_odom>true</publish_odom>
-      <publish_odom_tf>true</publish_odom_tf>
-      <publish_wheel_tf>true</publish_wheel_tf>
-    </plugin>
+      <plugin name="object_controller" filename="libgazebo_ros_planar_move.so">
+        <ros>
+          <argument>odom:=odom/unfiltered</argument>
+        </ros>
+        <command_topic>cmd_vel</command_topic>
+        <odometry_topic>odom/unfiltered</odometry_topic>
+        <odometry_frame>odom</odometry_frame>
+        <odometry_rate>20.0</odometry_rate>
+        <robot_base_frame>base_footprint</robot_base_frame>
+        <publish_odom>true</publish_odom>
+        <publish_odom_tf>false</publish_odom_tf>
+      </plugin>
+      <plugin name="robot_joint_state" filename="libgazebo_ros_joint_state_publisher.so">
+        <ros>
+          <remapping>joint_states:=joint_states</remapping>
+        </ros>
+        <update_rate>10</update_rate>
+        <joint_name>front_left_wheel_joint</joint_name>
+        <joint_name>front_right_wheel_joint</joint_name>
+        <joint_name>rear_left_wheel_joint</joint_name>
+        <joint_name>rear_right_wheel_joint</joint_name>
+      </plugin>
   </gazebo>
   </xacro:macro>

File: telerobot_description/urdf/mech/base.urdf.xacro (robot description, xacro)
@@ -8,5 +8,4 @@
         <geometry>
           <box size="${length} ${width} ${height}"/>
-          <!-- <mesh filename="" scale="0.001 0.001 0.001"/> -->
         </geometry>
         <material name="yellow">
@@ -20,11 +19,4 @@
         </geometry>
       </collision>
-      <inertial>
-        <origin xyz="0 0 0" rpy="0 0 0"/>
-        <mass value="${mass}"/>
-        <inertia ixx="${(1/12) * mass * ((width  * width)  + (height * height))}" ixy="0.0" ixz="0.0"
-                 iyy="${(1/12) * mass * ((length * length) + (height * height))}" iyz="0.0"
-                 izz="${(1/12) * mass * ((length * length) + (width  * width))}"/>
-      </inertial>
     </link>
     <gazebo reference="base_link">

File: telerobot_description/urdf/mech/mecanum_wheel.urdf.xacro (robot description, xacro)
@@ -18,11 +18,4 @@
         </geometry>
       </collision>
-      <inertial>
-        <origin xyz="0 0 0" rpy="0 0 0"/>
-        <mass value="${mass}"/>
-        <inertia ixx="${(2/5) * mass * (radius * radius)}" ixy="0" ixz="0"
-                 iyy="${(2/5) * mass * (radius * radius)}" iyz="0"
-                 izz="${(2/5) * mass * (radius * radius)}" />
-      </inertial>
     </link>
     <gazebo reference="${side}_wheel_link">

Commit message: Artem 3D model set.

File: telerobot_description/urdf/controllers/omni_drive.urdf.xacro (robot description, xacro)
@@ -2,26 +2,26 @@
   <xacro:macro name="omni_drive_controller">
     <gazebo>
-      <plugin name="object_controller" filename="libgazebo_ros_planar_move.so">
-        <ros>
-          <argument>odom:=odom/unfiltered</argument>
-        </ros>
-        <command_topic>cmd_vel</command_topic>
-        <odometry_topic>odom/unfiltered</odometry_topic>
-        <odometry_frame>odom</odometry_frame>
-        <odometry_rate>20.0</odometry_rate>
-        <robot_base_frame>base_footprint</robot_base_frame>
-        <publish_odom>true</publish_odom>
-        <publish_odom_tf>false</publish_odom_tf>
-      </plugin>
-      <plugin name="robot_joint_state" filename="libgazebo_ros_joint_state_publisher.so">
-        <ros>
-          <remapping>joint_states:=joint_states</remapping>
-        </ros>
-        <update_rate>10</update_rate>
-        <joint_name>front_left_wheel_joint</joint_name>
-        <joint_name>front_right_wheel_joint</joint_name>
-        <joint_name>rear_left_wheel_joint</joint_name>
-        <joint_name>rear_right_wheel_joint</joint_name>
-      </plugin>
+    <plugin name="object_controller" filename="libgazebo_ros_planar_move.so">
+      <ros>
+        <argument>odom:=odom/unfiltered</argument>
+      </ros>
+      <command_topic>cmd_vel</command_topic>
+      <odometry_topic>odom/unfiltered</odometry_topic>
+      <odometry_frame>odom</odometry_frame>
+      <odometry_rate>20.0</odometry_rate>
+      <robot_base_frame>base_footprint</robot_base_frame>
+      <publish_odom>true</publish_odom>
+      <publish_odom_tf>false</publish_odom_tf>
+    </plugin>
+    <plugin name="gazebo_joint_state" filename="libgazebo_ros_joint_state_publisher.so">
+      <ros>
+        <remapping>joint_states:=joint_states</remapping>
+      </ros>
+      <update_rate>30</update_rate>
+      <joint_name>front_left_wheel_joint</joint_name>
+      <joint_name>front_right_wheel_joint</joint_name>
+      <joint_name>rear_left_wheel_joint</joint_name>
+      <joint_name>rear_right_wheel_joint</joint_name>
+    </plugin>
   </gazebo>
   </xacro:macro>

File: telerobot_description/urdf/mech/base.urdf.xacro (robot description, xacro)
@@ -8,4 +8,5 @@
         <geometry>
           <box size="${length} ${width} ${height}"/>
+          <!-- <mesh filename="" scale="0.001 0.001 0.001"/> -->
         </geometry>
         <material name="yellow">
@@ -19,4 +20,11 @@
         </geometry>
       </collision>
+      <inertial>
+        <origin xyz="0 0 0" rpy="0 0 0"/>
+        <mass value="${mass}"/>
+        <inertia ixx="${(1/12) * mass * ((width  * width)  + (height * height))}" ixy="0.0" ixz="0.0"
+                 iyy="${(1/12) * mass * ((length * length) + (height * height))}" iyz="0.0"
+                 izz="${(1/12) * mass * ((length * length) + (width  * width))}"/>
+      </inertial>
     </link>
     <gazebo reference="base_link">

File: telerobot_description/urdf/mech/mecanum_wheel.urdf.xacro (robot description, xacro)
@@ -18,4 +18,11 @@
         </geometry>
       </collision>
+      <inertial>
+        <origin xyz="0 0 0" rpy="0 0 0"/>
+        <mass value="${mass}"/>
+        <inertia ixx="${(2/5) * mass * (radius * radius)}" ixy="0" ixz="0"
+                 iyy="${(2/5) * mass * (radius * radius)}" iyz="0"
+                 izz="${(2/5) * mass * (radius * radius)}" />
+      </inertial>
     </link>
     <gazebo reference="${side}_wheel_link">

File: telerobot_description/urdf/robots/telerobot.urdf.xacro (robot description, xacro)
@@ -14,5 +14,5 @@
     wheel_radius="${wheel_radius}"
     wheel_pos_z="${wheel_pos_z}"
-  />
+/>
   <xacro:mecanum_wheel
     side="front_left"

File: telerobot_description/urdf/sensors/generic_laser.urdf.xacro (robot description, xacro)
@@ -1,5 +1,5 @@
 <?xml version="1.0"?>
 <robot xmlns:xacro="http://ros.org/wiki/xacro">
-  <xacro:include filename="$(find linorobot2_description)/urdf/sensors/laser.urdf.xacro" />
+  <xacro:include filename="$(find telerobot_description)/urdf/sensors/laser.urdf.xacro" />
   <xacro:macro name="generic_laser" params="*origin">
     <xacro:laser

File: telerobot_description/urdf/sensors/laser.urdf.xacro (robot description, xacro)
@@ -36,4 +36,20 @@
       </visual>
     </gazebo>
+    <link name="laser_radius">
+      <visual>
+        <origin xyz="0 0 0" rpy="0 0 0"/>
+        <geometry>
+          <cylinder radius="0.1" length ="0.005"/>
+        </geometry>
+        <material name="blue">
+          <color rgba ="1 1 1 1"/>
+        </material>
+      </visual>
+    </link>
+    <joint name ="laser_radius_to_laser" type ="fixed">
+      <parent link="laser"/>
+      <child link="laser_radius"/>
+      <origin xyz="0 0 0" rpy="0 0 0"/>
+    </joint>
     <joint name="${frame_id}_to_base_link" type="fixed">
       <parent link="base_link"/>
