Commit message: Mikhalych

File: linorobot2_description/urdf/mecanum_properties.urdf.xacro (robot description, xacro)
@@ -13,5 +13,8 @@
   <xacro:property name="wheel_torque" value="20" />
   <xacro:property name="laser_pose">
-    <origin xyz="0.18 0 0.095" rpy="0 0 0"/>
+    <origin xyz="0.18 0.5 0.095" rpy="0 1.5707 0"/>
+  </xacro:property>
+  <xacro:property name="laser_pose1">
+    <origin xyz="-0.18 0.5 0.095" rpy="0 1.5707 0"/>
   </xacro:property>
   <xacro:property name="depth_sensor_pose">

File: linorobot2_description/urdf/robots/mecanum.urdf.xacro (robot description, xacro)
@@ -6,4 +6,5 @@
   <xacro:include filename="$(find linorobot2_description)/urdf/sensors/imu.urdf.xacro" />
   <xacro:include filename="$(find linorobot2_description)/urdf/sensors/generic_laser.urdf.xacro" />
+  <xacro:include filename="$(find linorobot2_description)/urdf/sensors/generic_laser1.urdf.xacro" />
   <xacro:include filename="$(find linorobot2_description)/urdf/sensors/depth_sensor.urdf.xacro" />
   <xacro:include filename="$(find linorobot2_description)/urdf/controllers/omni_drive.urdf.xacro" />
@@ -56,4 +57,7 @@
     <xacro:insert_block name="laser_pose" />
   </xacro:generic_laser>
+  <xacro:generic_laser1>
+    <xacro:insert_block name="laser_pose1" />
+  </xacro:generic_laser1>
   <!--<xacro:depth_sensor>
     <xacro:insert_block name="depth_sensor_pose" />

Commit message: remove Mikhalychs part

File: linorobot2_description/urdf/mecanum_properties.urdf.xacro (robot description, xacro)
@@ -13,8 +13,5 @@
   <xacro:property name="wheel_torque" value="20" />
   <xacro:property name="laser_pose">
-    <origin xyz="0.18 0.5 0.095" rpy="0 1.5707 0"/>
-  </xacro:property>
-  <xacro:property name="laser_pose1">
-    <origin xyz="-0.18 0.5 0.095" rpy="0 1.5707 0"/>
+    <origin xyz="0.18 0 0.095" rpy="0 0 0"/>
   </xacro:property>
   <xacro:property name="depth_sensor_pose">

File: linorobot2_description/urdf/robots/mecanum.urdf.xacro (robot description, xacro)
@@ -6,5 +6,4 @@
   <xacro:include filename="$(find linorobot2_description)/urdf/sensors/imu.urdf.xacro" />
   <xacro:include filename="$(find linorobot2_description)/urdf/sensors/generic_laser.urdf.xacro" />
-  <xacro:include filename="$(find linorobot2_description)/urdf/sensors/generic_laser1.urdf.xacro" />
   <xacro:include filename="$(find linorobot2_description)/urdf/sensors/depth_sensor.urdf.xacro" />
   <xacro:include filename="$(find linorobot2_description)/urdf/controllers/omni_drive.urdf.xacro" />
@@ -57,7 +56,4 @@
     <xacro:insert_block name="laser_pose" />
   </xacro:generic_laser>
-  <xacro:generic_laser1>
-    <xacro:insert_block name="laser_pose1" />
-  </xacro:generic_laser1>
   <!--<xacro:depth_sensor>
     <xacro:insert_block name="depth_sensor_pose" />

Commit message: remove Mikhalych

File: linorobot2_description/urdf/mecanum_properties.urdf.xacro (robot description, xacro)
@@ -13,8 +13,5 @@
   <xacro:property name="wheel_torque" value="20" />
   <xacro:property name="laser_pose">
-    <origin xyz="0.18 0.5 0.095" rpy="0 1.5707 0"/>
-  </xacro:property>
-  <xacro:property name="laser_pose1">
-    <origin xyz="-0.18 0.5 0.095" rpy="0 1.5707 0"/>
+    <origin xyz="0.18 0 0.095" rpy="0 0 0"/>
   </xacro:property>
   <xacro:property name="depth_sensor_pose">
